File: SilkscreenLinesText/SilkscreenLinesText.kicad_pcb (KiCad board)
At the start: 2 copper layers, 100 x 100 mm, 16 parts

Commit message: Updated header file reference, updated gerbers (zip, only)
Other:
- board text added: "${FILE} - ${LAYER}, rev ${REVISION}, issue ${ISSUE_DATE}"
- board text removed: "Lines.kicad_pcb - ${LAYER}, rev ${REVISION}, issue ${ISSUE_DATE}"
Changed lines of the file:
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@@
     )
   )
+  (property "FILE" "SilkscreenLinesText.kicad_pcb")
   (property "PCB_INFO" "Lines.kicad_pcb - ${LAYER}, rev ${REVISION}, issue ${ISSUE_DATE}")
   (net 0 "")
@@
   (gr_arc (start 51.335 41.195) (mid 52.799466 37.659466) (end 56.335 36.195)
     (stroke (width 0.1) (type default)) (layer "Edge.Cuts"))
-  (gr_text "Lines.kicad_pcb - ${LAYER}, rev ${REVISION}, issue ${ISSUE_DATE}" (at 139.335 37.195) (layer "B.SilkS")
+  (gr_text "${FILE} - ${LAYER}, rev ${REVISION}, issue ${ISSUE_DATE}" (at 139.335 37.195) (layer "B.SilkS")
     (effects (font (size 1 1) (thickness 0.15)) (justify left top mirror))
   )
-  (gr_text "Lines.kicad_pcb - ${LAYER}, rev ${REVISION}, issue ${ISSUE_DATE}" (at 63.335 37.195) (layer "F.SilkS")
+  (gr_text "${FILE} - ${LAYER}, rev ${REVISION}, issue ${ISSUE_DATE}" (at 63.335 37.195) (layer "F.SilkS")
     (effects (font (size 1 1) (thickness 0.15)) (justify left top))
   )
